File: Motion_potencia_2023/power/pcb_power.sch (EAGLE design)
At the start: 0 parts

Commit message: main, power
Parts:
- added 12V_OUT, 24V_L, 24V_MD, SWITCH1, SWITCH2, SWITCH3: 5566-25569-2, molex_arreglado_2:5566-25569-2
- added ADC_IN1, ADC_IN2, ADC_IN3, ADC_IN4, ADC_IN5: (no value), pinhead:PINHD-1X5
- added ADC_OUT1, ADC_OUT2, ADC_OUT3, ADC_OUT4, ADC_OUT5: (no value), pinhead:PINHD-1X4
- added AMP1, AMP2, AMP3, BUZZER: (no value), pinhead:PINHD-1X3
- added B1, B2, B4, B5: XT60-M, XT60-M:XT60-M
- added B1_A, B2_A, B3_A, B4_A, B5_A1, RASP: B4B-ZR, con-jst:B4B-ZR
- added B3: XT90, Robocol_Eagle_Libraries:XT90
- added B5_A: B5B-ZR(LF)(SN), B5B-ZR_LF__SN_:B5B-ZR(LF)(SN)
- added FUSE1, FUSE2: (no value), fuse:SHK20L
Connections:
- new net 5V: ADC_OUT1.4, ADC_OUT2.4, ADC_OUT3.4, ADC_OUT4.4, ADC_OUT5.4, AMP1.1, AMP2.1, AMP3.1, BUZZER.1, RASP-4.1
- new net AI1: ADC_IN1.2, B1_A-2.1
- new net AI10: ADC_IN3.3, B3_A-3.1
- new net AI11: ADC_IN3.4, B3_A-4.1
- new net AI12: ADC_IN3.5, AMP3.2
- new net AI13: ADC_IN4.2, B4_A-2.1
- new net AI14: ADC_IN4.3, B4_A-3.1
- new net AI15: ADC_IN4.4, B4_A-4.1
- new net AI16: ADC_IN4.5
- new net AI17: ADC_IN5.2, B5_A.2, B5_A1-2.1
- new net AI18: ADC_IN5.3, B5_A.3, B5_A1-3.1
- new net AI19: ADC_IN5.4, B5_A.4, B5_A1-4.1
- new net AI2: ADC_IN1.3, B1_A-3.1
- new net AI20: ADC_IN5.5, B5_A.5
- new net AI3: ADC_IN1.4, B1_A-4.1
- new net AI4: ADC_IN1.5, AMP1.2
- new net AI5: ADC_IN2.2, B2_A-2.1
- new net AI6: ADC_IN2.3, B2_A-3.1
- new net AI7: ADC_IN2.4, B2_A-4.1
- new net AI8: ADC_IN2.5, AMP2.2
- new net AI9: ADC_IN3.2, B3_A-2.1
- new net AO1: ADC_IN1.1, ADC_IN2.1, BUZZER.2
- new net GND: 12V_OUT-1.S, 24V_L-1.S, 24V_MD-1.S, ADC_OUT1.3, ADC_OUT2.3, ADC_OUT3.3, ADC_OUT4.3, ADC_OUT5.3, AMP1.3, AMP2.3, AMP3.3, B1_A-1.1, B2.NEG, B2_A-1.1, B3.-, B3_A-1.1, B4_A-1.1, B5.NEG, B5_A.1, B5_A1-1.1, BUZZER.3, RASP-1.1
- new net N$12: 24V_MD-2.S, FUSE1.1A, FUSE1.1B
- new net N$13: FUSE1.2A, FUSE1.2B, SWITCH2-2.S
- new net N$14: 12V_OUT-2.S, FUSE2.1A, FUSE2.1B
- new net N$15: FUSE2.2A, FUSE2.2B, SWITCH3-2.S
- new net N$16: 24V_L-2.S, SWITCH1-2.S
- new net N$17: B1.NEG, B2.POS
- new net N$20: B4.NEG, B5.POS
- new net SCL: ADC_OUT1.1, ADC_OUT2.1, ADC_OUT3.1, ADC_OUT4.1, ADC_OUT5.1, RASP-2.1
- new net SDAT: ADC_OUT1.2, ADC_OUT2.2, ADC_OUT3.2, ADC_OUT4.2, ADC_OUT5.2, RASP-3.1
- new net SWITCH1-1: B1.POS, SWITCH1-1.S
- new net SWITCH2-1: B3.+, SWITCH2-1.S
- new net SWITCH3-1: B4.POS, SWITCH3-1.S
Other:
- note added: "celda1 ADC1"
- note added: "celda2 ADC2"
- note added: "celda3 ADC3"
- note added: "celda4 ADC4"
- note added: "celda5 ADC5"
- note added: "perifericos auxiliares"
- note added: "salidas potencia e interrupciones"
- note added: "salidas rasp"
