File: Motion_potencia_2023/regulators/pcb_reguladores.sch (EAGLE design)
At the start: 19 parts, among them P1 USB-A1HSW6, X1 5566-25569-2, X3 5566-25569-2

Commit message: PCBs mandadas a fabricar
Changed lines of the file:
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@@
 <setting verticaltext="up"/>
 </settings>
-<grid distance="1" unitdist="mil" unit="mil" style="lines" multiple="1" display="no" altdistance="0.01" altunitdist="inch" altunit="inch"/>
+<grid distance="0.1" unitdist="inch" unit="inch" style="lines" multiple="1" display="no" altdistance="0.01" altunitdist="inch" altunit="inch"/>
 <layers>
 <layer number="1" name="Top" color="4" fill="1" visible="no" active="no"/>
@@
 <attribute name="VALUE" x="157.303" y="53.5084" size="1.778" layer="96"/>
 </instance>
-<instance part="X1" gate="-1" x="168.9108" y="98.8474" smashed="yes"/>
+<instance part="X1" gate="-1" x="113.0308" y="109.0074" smashed="yes"/>
 <instance part="X1" gate="-2" x="168.9108" y="93.7674" smashed="yes"/>
 <instance part="GND5" gate="1" x="165.8628" y="96.3074" smashed="yes">
@@
 <pinref part="X1" gate="-1" pin="S"/>
 <pinref part="GND5" gate="1" pin="GND"/>
-<wire x1="166.3708" y1="98.8474" x2="165.8628" y2="98.8474" width="0.1524" layer="91"/>
-</segment>
-<segment>
+<wire x1="110.4908" y1="109.0074" x2="165.8628" y2="98.8474" width="0.1524" layer="91"/>
+</segment>
+<segment>
